File: electronics/eeZeePower.sch (EAGLE design)
At the start: 11 parts

Commit message: converted to micro-B connector, shrunk board, changed layout to fit, modded silk slightly, removed 0.1uF output cap
Parts:
- removed C3: 0.1uF, rcl:C-USC0603
- removed U$1: USB-MINIB-5PIN, SparkFun:USB-MINIB-5PIN
- added JP1: USB-MICROB, SparkFun-Connectors:USB-MICROB
Connections:
- net GND: now also JP1.GND; no longer C3.2, U$1.GND, U$1.MTN1, U$1.MTN2, U$1.MTN3, U$1.MTN4
- net VBUS: now also JP1.VBUS; no longer U$1.VBUS
- net VOUT: no longer C3.1
