File: electronics/eeZeePower.sch (EAGLE design)
At the start: 11 parts

Commit message: replaced logo and document field.
Parts:
- added U$3: BOT-THOUGHTS-LOGO-MD, bt:BOT-THOUGHTS-LOGO-MD
Other:
- note added: "0.5"
- note removed: "0.4"
