File: electronics/eeZeePower.sch (EAGLE design)
At the start: 12 parts

Commit message: updated logo
Parts:
- removed U$3: BOT-THOUGHTS-LOGO-MD, bt:BOT-THOUGHTS-LOGO-MD
- added U$2: BTLOGO-LOGO-MD, bt:BTLOGO-LOGO-MD
Changed lines of the file:
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@@
 <part name="JP4" library="pinhead-2" deviceset="PINHD-1X02" device="_2.54-S"/>
 <part name="U$1" library="SparkFun" deviceset="USB-MINIB" device="-5PIN"/>
-<part name="U$3" library="bt" deviceset="BOT-THOUGHTS" device="-LOGO-MD" value="BOT-THOUGHTS-LOGO-MD"/>
 <part name="FRAME1" library="bt" deviceset="LETTER_L" device=""/>
+<part name="U$2" library="bt" deviceset="BTLOGO" device="-LOGO-MD" value="BTLOGO-LOGO-MD"/>
 </parts>
 <sheets>
@@
 <instance part="JP4" gate="A" x="182.88" y="129.54"/>
 <instance part="U$1" gate="G$1" x="55.88" y="109.22" rot="MR0"/>
-<instance part="U$3" gate="G$1" x="2.794" y="3.81"/>
 <instance part="FRAME1" gate="G$1" x="0" y="0"/>
 <instance part="FRAME1" gate="G$2" x="147.32" y="2.54"/>
+<instance part="U$2" gate="G$1" x="2.54" y="2.54"/>
 </instances>
 <busses>
